File: Slave/DifferentialSPIEncoder.sch (KiCad schematic (older format))
At the start: 31 parts, among them J1 Debug, J2 8P8C_LED_Shielded, U2 AS5048A, U3 SN65HVD06D, U4 SN65HVD06D, U5 SN65HVD06D

Commit message: Finish slave layout
Parts:
- J1: footprint Connector_PinHeader_2.54mm:PinHeader_1x06_P2.54mm_Vertical -> Connector_PinHeader_2.54mm:PinHeader_2x03_P2.54mm_Vertical
Changed lines of the file:
@@
 GND
-$Comp
-L Connector_Generic:Conn_02x03_Odd_Even J1
-U 1 1 5DE9B749
-P 7815 3175
-F 0 "J1" H 7865 3492 50  0000 C CNN
-F 1 "Debug" H 7865 3401 50  0000 C CNN
-F 2 "Connector_PinHeader_2.54mm:PinHeader_1x06_P2.54mm_Vertical" H 7815 3175 50  0001 C CNN
-F 3 "~" H 7815 3175 50  0001 C CNN
-	1    7815 3175
-	1    0    0    -1
-$EndComp
 $Comp
 L Mechanical:MountingHole H1
@@
 	1    0    0    -1
 $EndComp
+$Comp
+L Connector_Generic:Conn_02x03_Odd_Even J1
+U 1 1 5DE9B749
+P 7815 3175
+F 0 "J1" H 7865 3492 50  0000 C CNN
+F 1 "Debug" H 7865 3401 50  0000 C CNN
+F 2 "Connector_PinHeader_2.54mm:PinHeader_2x03_P2.54mm_Vertical" H 7815 3175 50  0001 C CNN
+F 3 "~" H 7815 3175 50  0001 C CNN
+	1    7815 3175
+	1    0    0    -1
+$EndComp
