File: Slave/DifferentialSPIEncoder.kicad_pcb (KiCad board)
At the start: 2 copper layers, 52.3 x 42.7 mm, 30 parts, among them J1 Debug, J2 8P8C_LED_Shielded, U1 AS5047U, U2 MAX14783ExS, U3 MAX14783ExS, U4 MAX14783ExS

Commit message: Finish encoder side layout
Parts:
- removed J2: 8P8C_LED_Shielded, Connector_RJ:RJ45_Amphenol_RJHSE538X
- removed R12, R13: 220, Resistor_SMD:R_0402_1005Metric
- added C3: 1uF, Capacitor_SMD:C_0603_1608Metric, F.Cu at (96.2, 98.5)
- added R1: 1k, Resistor_SMD:R_0603_1608Metric, F.Cu at (98.8, 93.8)
- added U5: MA702, Package_DFN_QFN:QFN-16-1EP_3x3mm_P0.5mm_EP1.8x1.8mm, F.Cu at (100.0, 100.0)
- C1: footprint Capacitor_SMD:C_0402_1005Metric -> Capacitor_SMD:C_0603_1608Metric; moved to F.Cu
- C2: moved to F.Cu
- C4, C5: value 2.2pF -> C; footprint Capacitor_SMD:C_0402_1005Metric -> Capacitor_SMD:C_0603_1608Metric
- C6: value 2.2pF -> 22nF; footprint Capacitor_SMD:C_0402_1005Metric -> Capacitor_SMD:C_0603_1608Metric
- C7, C8, C9: footprint Capacitor_SMD:C_0402_1005Metric -> Capacitor_SMD:C_0603_1608Metric; moved to B.Cu
- J1: value Debug -> RJ45_Shielded; footprint Connector_PinHeader_2.54mm:PinHeader_2x03_P2.54mm_Vertical -> Connector_RJ:RJ45_Amphenol_RJHSE5380; moved to B.Cu
- R10, R11, R8: footprint Resistor_SMD:R_0402_1005Metric -> Resistor_SMD:R_0603_1608Metric; moved to B.Cu
- R2: footprint Resistor_SMD:R_0402_1005Metric -> Resistor_SMD:R_0603_1608Metric
- R3: value 1k -> 10k; footprint Resistor_SMD:R_0402_1005Metric -> Resistor_SMD:R_0603_1608Metric
- R4: value 1k -> 10k; footprint Resistor_SMD:R_0402_1005Metric -> Resistor_SMD:R_0603_1608Metric; moved to B.Cu
- R5: value 10k -> 120; footprint Resistor_SMD:R_0402_1005Metric -> Resistor_SMD:R_0603_1608Metric; moved to B.Cu
- R6: value 10k -> 1k; footprint Resistor_SMD:R_0402_1005Metric -> Resistor_SMD:R_0603_1608Metric
- R7: value 10k -> 1k; footprint Resistor_SMD:R_0402_1005Metric -> Resistor_SMD:R_0603_1608Metric; moved to B.Cu
- R9: value 120 -> 10k; footprint Resistor_SMD:R_0402_1005Metric -> Resistor_SMD:R_0603_1608Metric; moved to B.Cu
- U1: value AS5047U -> AS5048A; moved to F.Cu
- U2, U3, U4: moved to B.Cu
- moved J1 33.5 mm to (96.2, 121.8), turned to 0 degrees
- moved R5 17.3 mm to (107.1, 112.5), turned to 180 degrees
- moved R10 15.9 mm to (92.8, 112.5)
- moved U2 15.1 mm to (107.1, 107.8)
- moved C8 13.7 mm to (89.3, 109.9), turned to 90 degrees
- moved C9 13.0 mm to (96.4, 109.9), turned to 90 degrees
- moved R8 12.2 mm to (92.2, 102.1), turned to 90 degrees
- moved U3 10.6 mm to (92.8, 107.8)
- moved R4 10.5 mm to (107.7, 102.1)
- moved U4 10.1 mm to (99.9, 107.8)
- moved R2 8.87 mm to (104.8, 95.5), turned to 180 degrees
- moved C7 8.82 mm to (103.5, 109.9), turned to 90 degrees
- moved R7 8.31 mm to (98.0, 102.1)
- moved C5 8.24 mm to (101.8, 93.8), turned to 90 degrees
- moved C4 7.79 mm to (104.8, 97.0), turned to 0 degrees
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Connections:
- C4 pad 1: ~CSn -> /~CSn
- C5 pad 1: CLK -> /CLK
- J1 pad 1: MISO -> (no net)
- J1 pad 3: CLK -> /CLK-
- J1 pad 4: /MOSI -> /MISO-
- J1 pad 5: ~CSn -> /MISO+
- J1 pad 6: GND -> /CLK+
- R10 pad 1: /CLK_- -> /MISO+
- R10 pad 2: /CLK_+ -> /MISO-
- R11 pad 1: /MISO_- -> /CLK+
- R11 pad 2: /MISO_+ -> /CLK-
- R2 pad 2: ~CSn -> /~CSn
- R3 pad 1: Net-(R3-Pad1) -> Net-(R2-Pad1)
- R3 pad 2: CLK -> +5V
- R4 pad 1: MISO -> GND
- R4 pad 2: Net-(C6-Pad1) -> Net-(R4-Pad2)
- R5 pad 1: Net-(R5-Pad1) -> /CS+
- R5 pad 2: GND -> /CS-
- R6 pad 1: +5V -> /MISO
- R6 pad 2: Net-(R2-Pad1) -> Net-(C6-Pad1)
- R7 pad 2: GND -> /CLK
- R8 pad 1: +5V -> Net-(R8-Pad1)
- R8 pad 2: Net-(R8-Pad2) -> +5V
- R9 pad 1: /CS_- -> GND
- R9 pad 2: /CS_+ -> Net-(R9-Pad2)
- U1 pad 1: ~CSn -> /~CSn
- U1 pad 10: Net-(U1-Pad10) -> (no net)
- U1 pad 14: /I -> (no net)
- U1 pad 2: CLK -> /CLK
- U1 pad 3: MISO -> /MISO
- U1 pad 4: /MOSI -> Net-(R1-Pad2)
- U1 pad 6: /B -> (no net)
- U1 pad 7: /A -> (no net)
- U1 pad 8: Net-(U1-Pad8) -> (no net)
- U1 pad 9: Net-(U1-Pad9) -> (no net)
- U2 pad 2: Net-(R7-Pad1) -> Net-(R4-Pad2)
- U2 pad 3: Net-(R7-Pad1) -> Net-(R4-Pad2)
- U2 pad 4: Net-(U2-Pad4) -> (no net)
- U2 pad 6: /CS_+ -> /CS+
- U2 pad 7: /CS_- -> /CS-
- U3 pad 1: Net-(U3-Pad1) -> (no net)
- U3 pad 2: Net-(R8-Pad2) -> Net-(R8-Pad1)
- U3 pad 3: Net-(R8-Pad2) -> Net-(R8-Pad1)
- U3 pad 6: /MISO_+ -> /MISO+
- U3 pad 7: /MISO_- -> /MISO-
- U4 pad 1: Net-(R3-Pad1) -> Net-(R7-Pad1)
- U4 pad 2: Net-(R5-Pad1) -> Net-(R9-Pad2)
- U4 pad 3: Net-(R5-Pad1) -> Net-(R9-Pad2)
- U4 pad 4: Net-(U4-Pad4) -> (no net)
- U4 pad 6: /CLK_+ -> /CLK+
- U4 pad 7: /CLK_- -> /CLK-
Routing:
- net GNDA: track 0.00 -> 29.7 mm
- net MISO: track 27.6 -> 0.00 mm, vias 2 -> 0
- net CLK: track 24.8 -> 0.00 mm, vias 1 -> 0
- net /CLK_+: track 18.8 -> 0.00 mm, vias 1 -> 0
- net /CLK_-: track 18.8 -> 0.00 mm, vias 1 -> 0
- net Net-(J2-PadSH): track 17.8 -> 0.00 mm
- net /CS_+: track 17.8 -> 0.00 mm
- net /CS_-: track 17.8 -> 0.00 mm
- net Net-(C6-Pad1): track 3.39 -> 20.6 mm, vias 0 -> 3
- net /MISO_-: track 16.3 -> 0.00 mm
- net /MISO_+: track 16.3 -> 0.00 mm
- net /MISO+: track 0.00 -> 14.3 mm
- net /CS-: track 0.00 -> 13.1 mm
- net ~CSn: track 12.9 -> 0.00 mm, vias 1 -> 0
- net /MISO-: track 0.00 -> 12.8 mm
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- added copper zone on F.Cu, net +5V
- added copper zone on B.Cu, net GND
- removed copper zone on B.Cu, net +5V
- removed copper zone on F.Cu, net GND
Other:
- board size 52.3 x 42.7 mm -> 52.3 x 45.7 mm
- board text added: "AS5048A Encoder Rev 3 2020-10-04"
- board text added: "https://github.com/Wetmelon"
- board text removed: "AS5048A Encoder Rev 2 2019-12-02"
- board text removed: "https://github.com/Wetmelon/DifferentialSPIEncoder"
