File: Slave/DifferentialSPIEncoder.kicad_sch (KiCad schematic)
At the start: 30 parts, among them J1 RJ45_Shielded, U1 AS5048A, U2 MAX14783ExS, U3 MAX14783ExS, U4 MAX14783ExS, U5 MA702

Commit message: Finish encoder side layout
Parts:
- C1, C2, C3, C4, C5, C6, C7, C8, C9: footprint Capacitor_SMD:C_0603_1608Metric_Pad1.05x0.95mm_HandSolder -> Capacitor_SMD:C_0603_1608Metric
- R1, R10, R11, R2, R3, R4, R5, R6, R7, R8, R9: footprint Resistor_SMD:R_0603_1608Metric_Pad1.05x0.95mm_HandSolder -> Resistor_SMD:R_0603_1608Metric
Connections:
- net +3V3: no longer R1.1
- net +5V: now also R1.1
