File: Master/DifferentialSPIMaster.sch (KiCad schematic (older format))
At the start: 37 parts, among them J1 Motor Encoder 0, J2 Conn_01x20, J3 Motor Encoder 0, U1 MAX485E, U2 MAX485E, U3 MAX485E, U4 MAX485E, U5 MAX485E, U6 MAX485E

Commit message: CLK is an output, not an input on master, also add edge cuts layer
Other:
- moved on the sheet: C10, C11, R11, R12
Changed lines of the file:
@@
 Wire Wire Line
 	6300 4750 6300 4700
-NoConn ~ 6700 4300
 Text Label 5400 4000 0    50   ~ 0
 CLK_1_-
@@
 L Device:R R12
 U 1 1 5D001624
-P 7300 4000
-F 0 "R12" V 7093 4000 50  0000 C CNN
-F 1 "R" V 7184 4000 50  0000 C CNN
-F 2 "Resistor_SMD:R_0805_2012Metric_Pad1.15x1.40mm_HandSolder" V 7230 4000 50  0001 C CNN
-F 3 "~" H 7300 4000 50  0001 C CNN
-	1    7300 4000
+P 7300 4300
+F 0 "R12" V 7093 4300 50  0000 C CNN
+F 1 "R" V 7184 4300 50  0000 C CNN
+F 2 "Resistor_SMD:R_0805_2012Metric_Pad1.15x1.40mm_HandSolder" V 7230 4300 50  0001 C CNN
+F 3 "~" H 7300 4300 50  0001 C CNN
+	1    7300 4300
 	0    -1   1    0
 $EndComp
@@
 L Device:C C11
 U 1 1 5D00162B
-P 7050 4250
-F 0 "C11" H 7165 4296 50  0000 L CNN
-F 1 "100nF" H 7165 4205 50  0000 L CNN
-F 2 "Capacitor_SMD:C_0805_2012Metric_Pad1.15x1.40mm_HandSolder" H 7088 4100 50  0001 C CNN
-F 3 "~" H 7050 4250 50  0001 C CNN
-	1    7050 4250
-	1    0    0    -1
-$EndComp
-Wire Wire Line
-	7050 4100 7050 4000
-Wire Wire Line
-	7050 4000 7150 4000
-Wire Wire Line
-	7050 4450 7050 4400
+P 7050 4550
+F 0 "C11" H 7165 4596 50  0000 L CNN
+F 1 "100nF" H 7165 4505 50  0000 L CNN
+F 2 "Capacitor_SMD:C_0805_2012Metric_Pad1.15x1.40mm_HandSolder" H 7088 4400 50  0001 C CNN
+F 3 "~" H 7050 4550 50  0001 C CNN
+	1    7050 4550
+	1    0    0    -1
+$EndComp
+Wire Wire Line
+	7050 4400 7050 4300
+Wire Wire Line
+	7050 4300 7150 4300
+Wire Wire Line
+	7050 4750 7050 4700
 $Comp
 L power:GNDD #PWR0111
 U 1 1 5D001635
-P 7050 4450
-F 0 "#PWR0111" H 7050 4200 50  0001 C CNN
-F 1 "GNDD" H 7054 4295 50  0001 C CNN
-F 2 "" H 7050 4450 50  0001 C CNN
-F 3 "" H 7050 4450 50  0001 C CNN
-	1    7050 4450
+P 7050 4750
+F 0 "#PWR0111" H 7050 4500 50  0001 C CNN
+F 1 "GNDD" H 7054 4595 50  0001 C CNN
+F 2 "" H 7050 4750 50  0001 C CNN
+F 3 "" H 7050 4750 50  0001 C CNN
+	1    7050 4750
 	-1   0    0    -1
 $EndComp
-Connection ~ 7050 4000
-Wire Wire Line
-	7800 4000 7450 4000
-Wire Wire Line
-	6700 4000 7050 4000
-Text Label 7800 4000 2    50   ~ 0
+Connection ~ 7050 4300
+Wire Wire Line
+	7800 4300 7450 4300
+Wire Wire Line
+	6700 4300 7050 4300
+Text Label 7800 4300 2    50   ~ 0
 SPI_SCK
 Wire Wire Line
@@
 Wire Wire Line
 	6200 10000 6200 9950
-NoConn ~ 6600 9550
 Text Label 5300 9250 0    50   ~ 0
 CLK_2_-
@@
 L Device:R R11
 U 1 1 5D027A7D
-P 7200 9250
-F 0 "R11" V 6993 9250 50  0000 C CNN
-F 1 "R" V 7084 9250 50  0000 C CNN
-F 2 "Resistor_SMD:R_0805_2012Metric_Pad1.15x1.40mm_HandSolder" V 7130 9250 50  0001 C CNN
-F 3 "~" H 7200 9250 50  0001 C CNN
-	1    7200 9250
+P 7200 9550
+F 0 "R11" V 6993 9550 50  0000 C CNN
+F 1 "R" V 7084 9550 50  0000 C CNN
+F 2 "Resistor_SMD:R_0805_2012Metric_Pad1.15x1.40mm_HandSolder" V 7130 9550 50  0001 C CNN
+F 3 "~" H 7200 9550 50  0001 C CNN
+	1    7200 9550
 	0    -1   1    0
 $EndComp
@@
 L Device:C C10
 U 1 1 5D027A84
-P 6950 9500
-F 0 "C10" H 7065 9546 50  0000 L CNN
-F 1 "100nF" H 7065 9455 50  0000 L CNN
-F 2 "Capacitor_SMD:C_0805_2012Metric_Pad1.15x1.40mm_HandSolder" H 6988 9350 50  0001 C CNN
-F 3 "~" H 6950 9500 50  0001 C CNN
-	1    6950 9500
-	1    0    0    -1
-$EndComp
-Wire Wire Line
-	6950 9350 6950 9250
-Wire Wire Line
-	6950 9250 7050 9250
-Wire Wire Line
-	6950 9700 6950 9650
+P 6950 9800
+F 0 "C10" H 7065 9846 50  0000 L CNN
+F 1 "100nF" H 7065 9755 50  0000 L CNN
+F 2 "Capacitor_SMD:C_0805_2012Metric_Pad1.15x1.40mm_HandSolder" H 6988 9650 50  0001 C CNN
+F 3 "~" H 6950 9800 50  0001 C CNN
+	1    6950 9800
+	1    0    0    -1
+$EndComp
+Wire Wire Line
+	6950 9650 6950 9550
+Wire Wire Line
+	6950 9550 7050 9550
+Wire Wire Line
+	6950 10000 6950 9950
 $Comp
 L power:GNDD #PWR0114
 U 1 1 5D027A8E
-P 6950 9700
-F 0 "#PWR0114" H 6950 9450 50  0001 C CNN
-F 1 "GNDD" H 6954 9545 50  0001 C CNN
-F 2 "" H 6950 9700 50  0001 C CNN
-F 3 "" H 6950 9700 50  0001 C CNN
-	1    6950 9700
+P 6950 10000
+F 0 "#PWR0114" H 6950 9750 50  0001 C CNN
+F 1 "GNDD" H 6954 9845 50  0001 C CNN
+F 2 "" H 6950 10000 50  0001 C CNN
+F 3 "" H 6950 10000 50  0001 C CNN
+	1    6950 10000
 	-1   0    0    -1
 $EndComp
-Connection ~ 6950 9250
-Wire Wire Line
-	7700 9250 7350 9250
-Wire Wire Line
-	6600 9250 6950 9250
+Connection ~ 6950 9550
+Wire Wire Line
+	7700 9550 7350 9550
+Wire Wire Line
+	6600 9550 6950 9550
 Wire Wire Line
 	3550 8650 3550 8700
@@
 Wire Wire Line
 	11350 4050 11750 4050
-Text Label 7700 9250 2    50   ~ 0
+Text Label 7700 9550 2    50   ~ 0
 SPI_SCK
 Wire Wire Line
@@
 L power:PWR_FLAG #FLG0104
 U 1 1 5DB973A9
-P 9550 1300
-F 0 "#FLG0104" H 9550 1375 50  0001 C CNN
-F 1 "PWR_FLAG" H 9550 1473 50  0000 C CNN
-F 2 "" H 9550 1300 50  0001 C CNN
-F 3 "~" H 9550 1300 50  0001 C CNN
-	1    9550 1300
-	1    0    0    -1
-$EndComp
-Wire Wire Line
-	9550 1300 9550 1350
-Wire Wire Line
-	9550 1350 9850 1350
+P 9800 1400
+F 0 "#FLG0104" H 9800 1475 50  0001 C CNN
+F 1 "PWR_FLAG" H 9800 1573 50  0000 C CNN
+F 2 "" H 9800 1400 50  0001 C CNN
+F 3 "~" H 9800 1400 50  0001 C CNN
+	1    9800 1400
+	1    0    0    -1
+$EndComp
+Wire Wire Line
+	9800 1400 9800 1450
+Wire Wire Line
+	9800 1450 10100 1450
 NoConn ~ 11750 2350
 NoConn ~ 11750 2450
@@
 $EndComp
 $Comp
-L power:+5V #PWR?
+L power:+5V #PWR0127
 U 1 1 5DA54465
-P 9850 1350
-F 0 "#PWR?" H 9850 1200 50  0001 C CNN
-F 1 "+5V" H 9865 1523 50  0000 C CNN
-F 2 "" H 9850 1350 50  0001 C CNN
-F 3 "" H 9850 1350 50  0001 C CNN
-	1    9850 1350
-	1    0    0    -1
-$EndComp
+P 10100 1450
+F 0 "#PWR0127" H 10100 1300 50  0001 C CNN
+F 1 "+5V" H 10115 1623 50  0000 C CNN
+F 2 "" H 10100 1450 50  0001 C CNN
+F 3 "" H 10100 1450 50  0001 C CNN
+	1    10100 1450
+	1    0    0    -1
+$EndComp
+NoConn ~ 6700 4000
+NoConn ~ 6600 9250
 $EndSCHEMATC

Commit message: Added values for LPFs
Parts:
- C10, C11, C2, C3, C5: value 100nF -> 2.2pF
- R11, R12, R14, R5, R8, R9: value R -> 1k
Other:
- note added: "LPF for single-ended signals:\nR = 680ohm\nC = 22pF\nFc = 10.6MHz"
Changed lines of the file:
@@
 encoding utf-8
 Sheet 1 1
-Title ""
-Date ""
-Rev ""
+Title "Differential SPI Encoder Master"
+Date "2019-11-06"
+Rev "2"
 Comp ""
 Comment1 ""
@@
 P 7100 2100
 F 0 "R5" V 6893 2100 50  0000 C CNN
-F 1 "R" V 6984 2100 50  0000 C CNN
+F 1 "1k" V 6984 2100 50  0000 C CNN
 F 2 "Resistor_SMD:R_0805_2012Metric_Pad1.15x1.40mm_HandSolder" V 7030 2100 50  0001 C CNN
 F 3 "~" H 7100 2100 50  0001 C CNN
@@
 P 7300 4300
 F 0 "R12" V 7093 4300 50  0000 C CNN
-F 1 "R" V 7184 4300 50  0000 C CNN
+F 1 "1k" V 7184 4300 50  0000 C CNN
 F 2 "Resistor_SMD:R_0805_2012Metric_Pad1.15x1.40mm_HandSolder" V 7230 4300 50  0001 C CNN
 F 3 "~" H 7300 4300 50  0001 C CNN
@@
 P 7050 4550
 F 0 "C11" H 7165 4596 50  0000 L CNN
-F 1 "100nF" H 7165 4505 50  0000 L CNN
+F 1 "2.2pF" H 7165 4505 50  0000 L CNN
 F 2 "Capacitor_SMD:C_0805_2012Metric_Pad1.15x1.40mm_HandSolder" H 7088 4400 50  0001 C CNN
 F 3 "~" H 7050 4550 50  0001 C CNN
@@
 P 7200 9550
 F 0 "R11" V 6993 9550 50  0000 C CNN
-F 1 "R" V 7084 9550 50  0000 C CNN
+F 1 "1k" V 7084 9550 50  0000 C CNN
 F 2 "Resistor_SMD:R_0805_2012Metric_Pad1.15x1.40mm_HandSolder" V 7130 9550 50  0001 C CNN
 F 3 "~" H 7200 9550 50  0001 C CNN
@@
 P 6950 9800
 F 0 "C10" H 7065 9846 50  0000 L CNN
-F 1 "100nF" H 7065 9755 50  0000 L CNN
+F 1 "2.2pF" H 7065 9755 50  0000 L CNN
 F 2 "Capacitor_SMD:C_0805_2012Metric_Pad1.15x1.40mm_HandSolder" H 6988 9650 50  0001 C CNN
 F 3 "~" H 6950 9800 50  0001 C CNN
@@
 P 4350 4300
 F 0 "R8" V 4143 4300 50  0000 C CNN
-F 1 "R" V 4234 4300 50  0000 C CNN
+F 1 "1k" V 4234 4300 50  0000 C CNN
 F 2 "Resistor_SMD:R_0805_2012Metric_Pad1.15x1.40mm_HandSolder" V 4280 4300 50  0001 C CNN
 F 3 "~" H 4350 4300 50  0001 C CNN
@@
 P 4100 4550
 F 0 "C3" H 4215 4596 50  0000 L CNN
-F 1 "100nF" H 4215 4505 50  0000 L CNN
+F 1 "2.2pF" H 4215 4505 50  0000 L CNN
 F 2 "Capacitor_SMD:C_0805_2012Metric_Pad1.15x1.40mm_HandSolder" H 4138 4400 50  0001 C CNN
 F 3 "~" H 4100 4550 50  0001 C CNN
@@
 P 4550 9550
 F 0 "R9" V 4343 9550 50  0000 C CNN
-F 1 "R" V 4434 9550 50  0000 C CNN
+F 1 "1k" V 4434 9550 50  0000 C CNN
 F 2 "Resistor_SMD:R_0805_2012Metric_Pad1.15x1.40mm_HandSolder" V 4480 9550 50  0001 C CNN
 F 3 "~" H 4550 9550 50  0001 C CNN
@@
 P 4300 9800
 F 0 "C5" H 4415 9846 50  0000 L CNN
-F 1 "100nF" H 4415 9755 50  0000 L CNN
+F 1 "2.2pF" H 4415 9755 50  0000 L CNN
 F 2 "Capacitor_SMD:C_0805_2012Metric_Pad1.15x1.40mm_HandSolder" H 4338 9650 50  0001 C CNN
 F 3 "~" H 4300 9800 50  0001 C CNN
@@
 P 9300 2350
 F 0 "C2" H 9415 2396 50  0000 L CNN
-F 1 "100nF" H 9415 2305 50  0000 L CNN
+F 1 "2.2pF" H 9415 2305 50  0000 L CNN
 F 2 "Capacitor_SMD:C_0805_2012Metric_Pad1.15x1.40mm_HandSolder" H 9338 2200 50  0001 C CNN
 F 3 "~" H 9300 2350 50  0001 C CNN
@@
 P 7000 7200
 F 0 "R14" V 6793 7200 50  0000 C CNN
-F 1 "R" V 6884 7200 50  0000 C CNN
+F 1 "1k" V 6884 7200 50  0000 C CNN
 F 2 "Resistor_SMD:R_0805_2012Metric_Pad1.15x1.40mm_HandSolder" V 6930 7200 50  0001 C CNN
 F 3 "~" H 7000 7200 50  0001 C CNN
@@
 NoConn ~ 6700 4000
 NoConn ~ 6600 9250
+Text Notes 7250 1200 0    75   ~ 0
+LPF for single-ended signals:\nR = 680ohm\nC = 22pF\nFc = 10.6MHz
 $EndSCHEMATC

Commit message: add BOM for parts
Parts:
- C1, C4, C6, C7, C8, C9: MANUFACTURER (none) -> KEMET; MFN (none) -> C0805C104K8RACTU
- C10, C11, C2, C3, C5: MANUFACTURER (none) -> KEMET; MFN (none) -> C0805C229C5GACTU
- J1, J3: MANUFACTURER (none) -> Amphenol Commercial Products; MFN (none) -> RJHSE5380
- R1, R13: MANUFACTURER (none) -> Yageo; MFN (none) -> AC0805JR-07120RL
- R10, R11, R12, R14, R2, R3, R4, R5, R6, R7, R8, R9: MANUFACTURER (none) -> Yageo; MFN (none) -> AC0805FR-7W1KL
- U1, U2, U3, U4, U5, U6: MANUFACTURER (none) -> Maxim Integrated; MFN (none) -> MAX485E

Commit message: Update master schematic with changes from #2
Parts:
- added R? (x4): 120, symbol Device:R_Small
- added R? (x2): 10k, Resistor_SMD:R_0805_2012Metric_Pad1.15x1.40mm_HandSolder, symbol Device:R
Connections:
- wire segments 147 -> 173
Other:
- moved on the sheet: C2, R14, R5

Commit message: Replace MAX485E with SN65HVD06D for 10mbps signaling
Parts:
- U1, U2, U3, U4, U5, U6: value MAX485E -> SN65HVD06D
Changed lines of the file:
@@
 P 6300 2200
 F 0 "U1" H 6100 2750 50  0000 C CNN
-F 1 "MAX485E" H 6100 2650 50  0000 C CNN
+F 1 "SN65HVD06D" H 6100 2650 50  0000 C CNN
 F 2 "Package_SO:SOIC-8_3.9x4.9mm_P1.27mm" H 6300 1500 50  0001 C CNN
 F 3 "https://www.mouser.com/ProductDetail/Maxim-Integrated/MAX485ESA%2b?qs=sGAEpiMZZMuXae9YOZoWd9EBnNihOkMOJLDcRh71%2FZA%3D" H 6300 2250 50  0001 C CNN
@@
 P 6300 4100
 F 0 "U3" H 6100 4650 50  0000 C CNN
-F 1 "MAX485E" H 6100 4550 50  0000 C CNN
+F 1 "SN65HVD06D" H 6100 4550 50  0000 C CNN
 F 2 "Package_SO:SOIC-8_3.9x4.9mm_P1.27mm" H 6300 3400 50  0001 C CNN
 F 3 "https://www.mouser.com/ProductDetail/Maxim-Integrated/MAX485ESA%2b?qs=sGAEpiMZZMuXae9YOZoWd9EBnNihOkMOJLDcRh71%2FZA%3D" H 6300 4150 50  0001 C CNN
@@
 P 6150 7300
 F 0 "U2" H 5950 7850 50  0000 C CNN
-F 1 "MAX485E" H 5950 7750 50  0000 C CNN
+F 1 "SN65HVD06D" H 5950 7750 50  0000 C CNN
 F 2 "Package_SO:SOIC-8_3.9x4.9mm_P1.27mm" H 6150 6600 50  0001 C CNN
 F 3 "https://www.mouser.com/ProductDetail/Maxim-Integrated/MAX485ESA%2b?qs=sGAEpiMZZMuXae9YOZoWd9EBnNihOkMOJLDcRh71%2FZA%3D" H 6150 7350 50  0001 C CNN
@@
 P 3550 4100
 F 0 "U4" H 3350 4650 50  0000 C CNN
-F 1 "MAX485E" H 3350 4550 50  0000 C CNN
+F 1 "SN65HVD06D" H 3350 4550 50  0000 C CNN
 F 2 "Package_SO:SOIC-8_3.9x4.9mm_P1.27mm" H 3550 3400 50  0001 C CNN
 F 3 "https://www.mouser.com/ProductDetail/Maxim-Integrated/MAX485ESA%2b?qs=sGAEpiMZZMuXae9YOZoWd9EBnNihOkMOJLDcRh71%2FZA%3D" H 3550 4150 50  0001 C CNN
@@
 P 6200 9350
 F 0 "U6" H 6000 9900 50  0000 C CNN
-F 1 "MAX485E" H 6000 9800 50  0000 C CNN
+F 1 "SN65HVD06D" H 6000 9800 50  0000 C CNN
 F 2 "Package_SO:SOIC-8_3.9x4.9mm_P1.27mm" H 6200 8650 50  0001 C CNN
 F 3 "https://www.mouser.com/ProductDetail/Maxim-Integrated/MAX485ESA%2b?qs=sGAEpiMZZMuXae9YOZoWd9EBnNihOkMOJLDcRh71%2FZA%3D" H 6200 9400 50  0001 C CNN
@@
 P 3550 9350
 F 0 "U5" H 3350 9900 50  0000 C CNN
-F 1 "MAX485E" H 3350 9800 50  0000 C CNN
+F 1 "SN65HVD06D" H 3350 9800 50  0000 C CNN
 F 2 "Package_SO:SOIC-8_3.9x4.9mm_P1.27mm" H 3550 8650 50  0001 C CNN
 F 3 "https://www.mouser.com/ProductDetail/Maxim-Integrated/MAX485ESA%2b?qs=sGAEpiMZZMuXae9YOZoWd9EBnNihOkMOJLDcRh71%2FZA%3D" H 3550 9400 50  0001 C CNN

Commit message: Add pullups for CS lines and remove extra material from master
Parts:
- R15, R16, R17, R18: renamed from R?; footprint (none) -> Resistor_SMD:R_0805_2012Metric_Pad1.15x1.40mm_HandSolder
- gave numbers to parts that had none: 2
Changed lines of the file:
@@
 LPF for single-ended signals:\nR = 680ohm\nC = 22pF\nFc = 10.6MHz
 $Comp
-L Device:R_Small R?
+L Device:R_Small R15
 U 1 1 5DE50CE4
 P 2950 4150
-F 0 "R?" H 2891 4196 50  0000 R CNN
+F 0 "R15" H 2891 4196 50  0000 R CNN
 F 1 "120" H 2891 4105 50  0000 R CNN
-F 2 "" H 2950 4150 50  0001 C CNN
+F 2 "Resistor_SMD:R_0805_2012Metric_Pad1.15x1.40mm_HandSolder" H 2950 4150 50  0001 C CNN
 F 3 "~" H 2950 4150 50  0001 C CNN
 	1    2950 4150
@@
 	2950 4300 3150 4300
 $Comp
-L Device:R_Small R?
+L Device:R_Small R18
 U 1 1 5DE7136E
 P 5750 4150
-F 0 "R?" H 5691 4196 50  0000 R CNN
+F 0 "R18" H 5691 4196 50  0000 R CNN
 F 1 "120" H 5691 4105 50  0000 R CNN
-F 2 "" H 5750 4150 50  0001 C CNN
+F 2 "Resistor_SMD:R_0805_2012Metric_Pad1.15x1.40mm_HandSolder" H 5750 4150 50  0001 C CNN
 F 3 "~" H 5750 4150 50  0001 C CNN
 	1    5750 4150
@@
 	5750 4300 5900 4300
 $Comp
-L Device:R_Small R?
+L Device:R_Small R16
 U 1 1 5DE7E37C
 P 2950 9400
-F 0 "R?" H 2891 9446 50  0000 R CNN
+F 0 "R16" H 2891 9446 50  0000 R CNN
 F 1 "120" H 2891 9355 50  0000 R CNN
-F 2 "" H 2950 9400 50  0001 C CNN
+F 2 "Resistor_SMD:R_0805_2012Metric_Pad1.15x1.40mm_HandSolder" H 2950 9400 50  0001 C CNN
 F 3 "~" H 2950 9400 50  0001 C CNN
 	1    2950 9400
@@
 	2950 9550 3150 9550
 $Comp
-L Device:R_Small R?
+L Device:R_Small R17
 U 1 1 5DE9AF13
 P 5650 9400
-F 0 "R?" H 5591 9446 50  0000 R CNN
+F 0 "R17" H 5591 9446 50  0000 R CNN
 F 1 "120" H 5591 9355 50  0000 R CNN
-F 2 "" H 5650 9400 50  0001 C CNN
+F 2 "Resistor_SMD:R_0805_2012Metric_Pad1.15x1.40mm_HandSolder" H 5650 9400 50  0001 C CNN
 F 3 "~" H 5650 9400 50  0001 C CNN
 	1    5650 9400
@@
 	5650 9550 5800 9550
 $Comp
-L Device:R R?
+L Device:R R19
 U 1 1 5DEB92EB
 P 6700 6950
-F 0 "R?" H 6770 6996 50  0000 L CNN
+F 0 "R19" H 6770 6996 50  0000 L CNN
 F 1 "10k" H 6770 6905 50  0000 L CNN
 F 2 "Resistor_SMD:R_0805_2012Metric_Pad1.15x1.40mm_HandSolder" V 6630 6950 50  0001 C CNN
@@
 	6150 6650 6150 6800
 $Comp
-L Device:R R?
+L Device:R R20
 U 1 1 5DED04F7
 P 6850 1850
-F 0 "R?" H 6920 1896 50  0000 L CNN
+F 0 "R20" H 6920 1896 50  0000 L CNN
 F 1 "10k" H 6920 1805 50  0000 L CNN
 F 2 "Resistor_SMD:R_0805_2012Metric_Pad1.15x1.40mm_HandSolder" V 6780 1850 50  0001 C CNN

Commit message: Swap to MAX14783E
Parts:
- removed U1, U2, U3, U4, U5, U6: SN65HVD06D, Package_SO:SOIC-8_3.9x4.9mm_P1.27mm, symbol Interface_UART:MAX485E
- added U1, U2, U3, U4, U5: MAX14783ExS, Package_SO:SOIC-8_3.9x4.9mm_P1.27mm, symbol Interface_UART:MAX14783ExS
Changed lines of the file:
@@
 EESchema Schematic File Version 4
-LIBS:DifferentialSPIMaster-cache
 EELAYER 30 0
 EELAYER END
@@
 MISO_1_+
 $Comp
-L Interface_UART:MAX485E U1
-U 1 1 5CF3CC79
-P 6300 2200
-F 0 "U1" H 6100 2750 50  0000 C CNN
-F 1 "SN65HVD06D" H 6100 2650 50  0000 C CNN
-F 2 "Package_SO:SOIC-8_3.9x4.9mm_P1.27mm" H 6300 1500 50  0001 C CNN
-F 3 "https://www.mouser.com/ProductDetail/Maxim-Integrated/MAX485ESA%2b?qs=sGAEpiMZZMuXae9YOZoWd9EBnNihOkMOJLDcRh71%2FZA%3D" H 6300 2250 50  0001 C CNN
-F 4 "Maxim Integrated" H 6300 2200 50  0001 C CNN "MANUFACTURER"
-F 5 "MAX485E" H 6300 2200 50  0001 C CNN "MFN"
-	1    6300 2200
-	-1   0    0    -1
-$EndComp
-$Comp
 L Connector:8P8C_Shielded J1
 U 1 1 5CF3CBE0
@@
 CLK_1_+
 $Comp
-L Interface_UART:MAX485E U3
-U 1 1 5D026421
-P 6300 4100
-F 0 "U3" H 6100 4650 50  0000 C CNN
-F 1 "SN65HVD06D" H 6100 4550 50  0000 C CNN
-F 2 "Package_SO:SOIC-8_3.9x4.9mm_P1.27mm" H 6300 3400 50  0001 C CNN
-F 3 "https://www.mouser.com/ProductDetail/Maxim-Integrated/MAX485ESA%2b?qs=sGAEpiMZZMuXae9YOZoWd9EBnNihOkMOJLDcRh71%2FZA%3D" H 6300 4150 50  0001 C CNN
-F 4 "Maxim Integrated" H 6300 4100 50  0001 C CNN "MANUFACTURER"
-F 5 "MAX485E" H 6300 4100 50  0001 C CNN "MFN"
-	1    6300 4100
-	-1   0    0    -1
-$EndComp
-$Comp
 L power:GNDD #PWR08
 U 1 1 5D026428
@@
 MISO_2_-
 $Comp
-L Interface_UART:MAX485E U2
-U 1 1 5CFD4CEE
-P 6150 7300
-F 0 "U2" H 5950 7850 50  0000 C CNN
-F 1 "SN65HVD06D" H 5950 7750 50  0000 C CNN
-F 2 "Package_SO:SOIC-8_3.9x4.9mm_P1.27mm" H 6150 6600 50  0001 C CNN
-F 3 "https://www.mouser.com/ProductDetail/Maxim-Integrated/MAX485ESA%2b?qs=sGAEpiMZZMuXae9YOZoWd9EBnNihOkMOJLDcRh71%2FZA%3D" H 6150 7350 50  0001 C CNN
-F 4 "Maxim Integrated" H 6150 7300 50  0001 C CNN "MANUFACTURER"
-F 5 "MAX485E" H 6150 7300 50  0001 C CNN "MFN"
-	1    6150 7300
-	-1   0    0    -1
-$EndComp
-$Comp
 L power:GNDD #PWR0104
 U 1 1 5CFD4CF5
@@
 Text Label 2600 4000 0    50   ~ 0
 CS_1_-
-$Comp
-L Interface_UART:MAX485E U4
-U 1 1 5CFD62E4
-P 3550 4100
-F 0 "U4" H 3350 4650 50  0000 C CNN
-F 1 "SN65HVD06D" H 3350 4550 50  0000 C CNN
-F 2 "Package_SO:SOIC-8_3.9x4.9mm_P1.27mm" H 3550 3400 50  0001 C CNN
-F 3 "https://www.mouser.com/ProductDetail/Maxim-Integrated/MAX485ESA%2b?qs=sGAEpiMZZMuXae9YOZoWd9EBnNihOkMOJLDcRh71%2FZA%3D" H 3550 4150 50  0001 C CNN
-F 4 "Maxim Integrated" H 3550 4100 50  0001 C CNN "MANUFACTURER"
-F 5 "MAX485E" H 3550 4100 50  0001 C CNN "MFN"
-	1    3550 4100
-	-1   0    0    -1
-$EndComp
 $Comp
 L power:GNDD #PWR0106
@@
 CLK_2_+
 $Comp
-L Interface_UART:MAX485E U6
-U 1 1 5D027A5E
-P 6200 9350
-F 0 "U6" H 6000 9900 50  0000 C CNN
-F 1 "SN65HVD06D" H 6000 9800 50  0000 C CNN
-F 2 "Package_SO:SOIC-8_3.9x4.9mm_P1.27mm" H 6200 8650 50  0001 C CNN
-F 3 "https://www.mouser.com/ProductDetail/Maxim-Integrated/MAX485ESA%2b?qs=sGAEpiMZZMuXae9YOZoWd9EBnNihOkMOJLDcRh71%2FZA%3D" H 6200 9400 50  0001 C CNN
-F 4 "Maxim Integrated" H 6200 9350 50  0001 C CNN "MANUFACTURER"
-F 5 "MAX485E" H 6200 9350 50  0001 C CNN "MFN"
-	1    6200 9350
-	-1   0    0    -1
-$EndComp
-$Comp
 L power:GNDD #PWR0113
 U 1 1 5D027A65
@@
 Text Label 2400 9250 0    50   ~ 0
 CS_2_-
-$Comp
-L Interface_UART:MAX485E U5
-U 1 1 5D030238
-P 3550 9350
-F 0 "U5" H 3350 9900 50  0000 C CNN
-F 1 "SN65HVD06D" H 3350 9800 50  0000 C CNN
-F 2 "Package_SO:SOIC-8_3.9x4.9mm_P1.27mm" H 3550 8650 50  0001 C CNN
-F 3 "https://www.mouser.com/ProductDetail/Maxim-Integrated/MAX485ESA%2b?qs=sGAEpiMZZMuXae9YOZoWd9EBnNihOkMOJLDcRh71%2FZA%3D" H 3550 9400 50  0001 C CNN
-F 4 "Maxim Integrated" H 3550 9350 50  0001 C CNN "MANUFACTURER"
-F 5 "MAX485E" H 3550 9350 50  0001 C CNN "MFN"
-	1    3550 9350
-	-1   0    0    -1
-$EndComp
 $Comp
 L power:GNDD #PWR0116
@@
 Wire Wire Line
 	6850 2200 6700 2200
+$Comp
+L Interface_UART:MAX14783ExS U4
+U 1 1 5F1861DC
+P 6300 2200
+F 0 "U4" H 6300 2881 50  0000 C CNN
+F 1 "MAX14783ExS" H 6300 2790 50  0000 C CNN
+F 2 "Package_SO:SOIC-8_3.9x4.9mm_P1.27mm" H 6300 1300 50  0001 C CNN
+F 3 "https://datasheets.maximintegrated.com/en/ds/MAX14783E.pdf" H 6300 2250 50  0001 C CNN
+	1    6300 2200
+	-1   0    0    -1
+$EndComp
+$Comp
+L Interface_UART:MAX14783ExS U5
+U 1 1 5F188E05
+P 6300 4100
+F 0 "U5" H 6300 4781 50  0000 C CNN
+F 1 "MAX14783ExS" H 6300 4690 50  0000 C CNN
+F 2 "Package_SO:SOIC-8_3.9x4.9mm_P1.27mm" H 6300 3200 50  0001 C CNN
+F 3 "https://datasheets.maximintegrated.com/en/ds/MAX14783E.pdf" H 6300 4150 50  0001 C CNN
+	1    6300 4100
+	-1   0    0    -1
+$EndComp
+$Comp
+L Interface_UART:MAX14783ExS U1
+U 1 1 5F189A10
+P 3550 4100
+F 0 "U1" H 3550 4781 50  0000 C CNN
+F 1 "MAX14783ExS" H 3550 4690 50  0000 C CNN
+F 2 "Package_SO:SOIC-8_3.9x4.9mm_P1.27mm" H 3550 3200 50  0001 C CNN
+F 3 "https://datasheets.maximintegrated.com/en/ds/MAX14783E.pdf" H 3550 4150 50  0001 C CNN
+	1    3550 4100
+	-1   0    0    -1
+$EndComp
+$Comp
+L Interface_UART:MAX14783ExS U3
+U 1 1 5F18B868
+P 6200 9350
+F 0 "U3" H 6200 10031 50  0000 C CNN
+F 1 "MAX14783ExS" H 6200 9940 50  0000 C CNN
+F 2 "Package_SO:SOIC-8_3.9x4.9mm_P1.27mm" H 6200 8450 50  0001 C CNN
+F 3 "https://datasheets.maximintegrated.com/en/ds/MAX14783E.pdf" H 6200 9400 50  0001 C CNN
+	1    6200 9350
+	-1   0    0    -1
+$EndComp
+$Comp
+L Interface_UART:MAX14783ExS U2
+U 1 1 5F18E086
+P 3550 9350
+F 0 "U2" H 3550 10031 50  0000 C CNN
+F 1 "MAX14783ExS" H 3550 9940 50  0000 C CNN
+F 2 "Package_SO:SOIC-8_3.9x4.9mm_P1.27mm" H 3550 8450 50  0001 C CNN
+F 3 "https://datasheets.maximintegrated.com/en/ds/MAX14783E.pdf" H 3550 9400 50  0001 C CNN
+	1    3550 9350
+	-1   0    0    -1
+$EndComp
 $EndSCHEMATC
