File: Master/DifferentialSPIMaster.sch (KiCad schematic (older format))
At the start: 43 parts, among them J1 Motor Encoder 0, J2 Conn_01x20, J3 Motor Encoder 0, U1 MAX14783ExS, U2 MAX14783ExS, U3 MAX14783ExS, U4 MAX14783ExS, U5 MAX14783ExS, U6 MAX14783ExS

Commit message: Update master
Parts:
- removed C1, C4, C6, C7, C8, C9: 100nF, Capacitor_SMD:C_0805_2012Metric_Pad1.15x1.40mm_HandSolder, symbol Device:C
- removed C10, C11, C3, C5: 2.2pF, Capacitor_SMD:C_0805_2012Metric_Pad1.15x1.40mm_HandSolder, symbol Device:C
- removed J1, J3: Motor Encoder 0, Connector_RJ:RJ45_Amphenol_RJHSE5380, symbol Connector:8P8C_Shielded
- removed J2: Conn_01x20, Connector_PinHeader_2.54mm:PinHeader_1x20_P2.54mm_Vertical, symbol Connector_Generic:Conn_01x20
- removed R10, R11, R12, R14, R2, R3, R4, R5, R6, R7, R8, R9: 1k, Resistor_SMD:R_0805_2012Metric_Pad1.15x1.40mm_HandSolder, symbol Device:R
- removed R19, R20: 10k, Resistor_SMD:R_0805_2012Metric_Pad1.15x1.40mm_HandSolder, symbol Device:R
- added C1, C10, C11, C3: C_Small, Capacitor_SMD:C_0805_2012Metric_Pad1.15x1.40mm_HandSolder, symbol Device:C_Small
- added C4, C5, C6, C7, C8, C9: 100nF, Capacitor_SMD:C_0805_2012Metric_Pad1.15x1.40mm_HandSolder, symbol Device:C_Small
- added J1, J2: RJ45_Shielded, Connector_RJ:RJ45_Amphenol_RJHSE5380, symbol Connector:RJ45_Shielded
- added J3: Conn_01x20, Connector_PinSocket_2.54mm:PinSocket_1x20_P2.54mm_Vertical, symbol Connector_Generic:Conn_01x20
- added R10, R2, R7, R8, R9: 120, Resistor_SMD:R_0805_2012Metric_Pad1.15x1.40mm_HandSolder, symbol Device:R_Small
- added R11, R12, R14, R3, R4: R_Small, Resistor_SMD:R_0805_2012Metric_Pad1.15x1.40mm_HandSolder, symbol Device:R_Small
- added R19, R20, R5, R6: 1k, Resistor_SMD:R_0805_2012Metric_Pad1.15x1.40mm_HandSolder, symbol Device:R_Small
- R1: MANUFACTURER Yageo -> (none); MFN AC0805JR-07120RL -> (none)
- R13: value 120 -> 1k; MANUFACTURER Yageo -> (none); MFN AC0805JR-07120RL -> (none)
- R15, R17, R18: value 120 -> 1k
- R16: value 120 -> R_Small
Connections:
- net labels added: GNDA, SPI_MOSI
- wire segments 173 -> 172
- no-connect marks 17 -> 16
Other:
- moved on the sheet: C2, NT1
